Commit message: fix spawn 2 robots with xacro and gazebo

File: my_box_bot_description/urdf/box_bot.gazebo.xacro (robot description, xacro)
@@ -1,5 +1,4 @@
 <?xml version="1.0"?>
 <robot xmlns:xacro="http://www.ros.org/wiki/xacro">
-<xacro:property name="robot_name" value="$(arg robot_name)"/>
 <xacro:macro name="gazebo_elements">
   <gazebo reference="left_wheel">
@@ -43,5 +42,6 @@
     <material>Gazebo/Red</material>
   </gazebo>
-  <gazebo>
+</xacro:macro>
+<gazebo>
     <plugin name="box_bot_joint_state" filename="libgazebo_ros_joint_state_publisher.so">
       <ros>
@@ -84,4 +84,3 @@
     </plugin>
   </gazebo>
-</xacro:macro>
 </robot>

File: my_box_bot_description/urdf/box_bot.xacro (robot description, xacro)
@@ -1,5 +1,10 @@
 <?xml version="1.0"?>
 <robot xmlns:xacro="http://www.ros.org/wiki/xacro" name="my_box_bot">
-<xacro:include filename="$(find my_box_bot_description)/urdf/box_bot.gazebo.xacro" />
+<xacro:property name="robot_name" value="$(arg robot_name)"/>
+<xacro:arg name="use_sim" default="true" />
+<!-- if we use Gazebo -->
+<xacro:if value="$(arg use_sim)">
+    <xacro:include filename="$(find my_box_bot_description)/urdf/box_bot.gazebo.xacro" />
+</xacro:if>
 <xacro:property name="body_width" value="0.1"/>
 <xacro:property name="body_lenght" value="0.1"/>
@@ -202,4 +207,5 @@
       </inertial>
   </link>
+Exercise
   <joint name="back_roll_joint" type="continuous">
     <origin rpy="0 0 0" xyz="0 0 0" />
